File: KiCad-projects/Buzzer-game-client/Buzzer-Client.kicad_sch (KiCad schematic)
At the start: 9 parts, among them SW1 SW_Push, SW2 SW_DPST_x2, U2 NRF24L01_Breakout

Commit message: skeem+pins
Other:
- note added: "Button pins"
- note added: "btn1"
- note added: "btn2"
- note added: "led1"
- note added: "led2"
Changed lines of the file:
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@@
+		)
+	)
+	(circle
+		(center 255.016 142.494)
+		(radius 1.27)
+		(stroke
+			(width 0)
+			(type default)
+		)
+		(fill
+			(type none)
+		)
+	)
+	(rectangle
+		(start 224.536 108.204)
+		(end 277.876 159.004)
+		(stroke
+			(width 0)
+			(type default)
+		)
+		(fill
+			(type none)
+		)
+	)
+	(rectangle
+		(start 252.476 151.384)
+		(end 257.556 156.464)
+		(stroke
+			(width 0)
+			(type default)
+		)
+		(fill
+			(type color)
+			(color 255 255 194 1)
+		)
+	)
+	(rectangle
+		(start 238.506 134.874)
+		(end 247.396 139.954)
+		(stroke
+			(width 0)
+			(type default)
+		)
+		(fill
+			(type color)
+			(color 255 255 194 1)
+		)
+	)
+	(rectangle
+		(start 262.636 134.874)
+		(end 271.526 139.954)
+		(stroke
+			(width 0)
+			(type default)
+		)
+		(fill
+			(type color)
+			(color 255 255 194 1)
+		)
+	)
+	(circle
+		(center 255.016 153.924)
+		(radius 1.27)
+		(stroke
+			(width 0)
+			(type default)
+		)
+		(fill
+			(type none)
+		)
+	)
+	(rectangle
+		(start 252.476 131.064)
+		(end 257.556 145.034)
+		(stroke
+			(width 0)
+			(type default)
+		)
+		(fill
+			(type color)
+			(color 255 255 194 1)
 		)
 	)
@@
 		)
 	)
+	(circle
+		(center 241.046 137.414)
+		(radius 1.27)
+		(stroke
+			(width 0)
+			(type default)
+		)
+		(fill
+			(type none)
+		)
+	)
+	(circle
+		(center 268.986 137.16)
+		(radius 1.27)
+		(stroke
+			(width 0)
+			(type default)
+		)
+		(fill
+			(type none)
+		)
+	)
+	(rectangle
+		(start 247.396 120.904)
+		(end 262.636 151.384)
+		(stroke
+			(width 0)
+			(type default)
+		)
+		(fill
+			(type none)
+		)
+	)
 	(text "nRF24L01"
 		(exclude_from_sim no)
@@
 		(effects
 			(font
-				(size 2 2)
-			)
-			(justify left bottom)
+				(size 2.54 2.54)
+			)
+			(justify left bottom)
+		)
+	)
+	(text "led2"
+		(exclude_from_sim no)
+		(at 268.986 132.334 0)
+		(effects
+			(font
+				(size 1.27 1.27)
+			)
 		)
 	)
 	(text "Main button\nand LED"
 		(exclude_from_sim no)
-		(at 26.162 55.88 0)
-		(effects
-			(font
-				(size 2 2)
-			)
-			(justify left bottom)
+		(at 21.082 58.674 0)
+		(effects
+			(font
+				(size 2.54 2.54)
+			)
+			(justify left bottom)
+		)
+	)
+	(text "led1"
+		(exclude_from_sim no)
+		(at 240.792 132.588 0)
+		(effects
+			(font
+				(size 1.27 1.27)
+			)
+		)
+	)
+	(text "btn1"
+		(exclude_from_sim no)
+		(at 260.35 143.256 0)
+		(effects
+			(font
+				(size 1.27 1.27)
+			)
+		)
+	)
+	(text "btn2"
+		(exclude_from_sim no)
+		(at 260.35 155.448 0)
+		(effects
+			(font
+				(size 1.27 1.27)
+			)
 		)
 	)
@@
 		(effects
 			(font
-				(size 2 2)
-			)
-			(justify left bottom)
+				(size 2.54 2.54)
+			)
+			(justify left bottom)
+		)
+	)
+	(text "Button pins"
+		(exclude_from_sim no)
+		(at 240.03 115.57 0)
+		(effects
+			(font
+				(size 2.54 2.54)
+			)
 		)
 	)
@@
 		(effects
 			(font
-				(size 2 2)
-			)
-			(justify left bottom)
+				(size 2.54 2.54)
+			)
+			(justify left bottom)
