File: KiCad-projects/Buzzer-game-server/Buzzer-Server.kicad_sch (KiCad schematic)
At the start: 9 parts, among them Q1 PN2222A, SW1 SW_Push, SW2 SW_DPST_x2, U1 Pico

Commit message: skeem+pins
Parts:
- removed Q1: PN2222A, Package_TO_SOT_THT:TO-92_Inline, symbol Transistor_BJT:PN2222A
- added D2: Player 1 LED, symbol Device:LED
- added D3: Player 2 LED, symbol Device:LED
- added D4: Player 3 LED, symbol Device:LED
- added D5: Player 4 LED, symbol Device:LED
- added D6: Status LED, symbol Device:LED
- added R4, R5, R6, R7, R8: R, symbol Device:R
- added SW3: SW_Push, symbol Switch:SW_Push
- added U2: NRF24L01_Breakout, RF_Module:nRF24L01_Breakout, symbol RF:NRF24L01_Breakout
- BT1: value Battery -> Battery 4xAA
- D1: value MAIN LED -> Player 0 LED
Connections:
- net LED_4_PIN is gone; now on net Ready BTN: U1.12 (GPIO9)
- net LED_5_PIN is gone; now on net Player_0: U1.14 (GPIO10)
- net 3V3: now also R1.1, R3.1, U2.2 (VCC); no longer SW1.1
- net GND: now also D1.1 (K), SW1.1, U1.23 (GND), D2.1 (K), D3.1 (K), D4.1 (K), D5.1 (K), D6.1 (K), SW3.1, U2.1 (GND); no longer R3.2, U1.13 (GND), U1.8 (GND)
- net Player_0: now reaches R2.1
- net Player_0: no longer D1.1 (K)
- net at R2.2: now also D1.2 (A)
- net Player_1: now reaches U1.15 (GPIO11)
- net Player_1: now also R4.1
- net Player_2: now reaches U1.16 (GPIO12)
- net Player_2: now also R5.1
- net Player_3: now reaches U1.17 (GPIO13)
- net Player_3: now also R6.1
- net Status: now reaches U1.20 (GPIO15)
- net Status: now also R8.1
- net CSN: now reaches U1.21 (GPIO16)
- net CSN: now also U2.4 (~{CSN})
- net CE: now reaches U1.22 (GPIO17)
- net CE: now also U2.3 (CE)
- net SCK: now reaches U1.24 (GPIO18)
- net SCK: now also U2.5 (SCK)
- net MOSI: now reaches U1.25 (GPIO19)
- net MOSI: now also U2.6 (MOSI)
- net MISO: now reaches U1.26 (GPIO20)
- net MISO: now also U2.7 (MISO)
- net Ready BTN: now reaches R1.2
- net Ready BTN: now also SW3.2
- removed net BTN_RESET_PIN: R3.1, SW1.2, U1.4 (GPIO2)
- net BTN_START_PIN: no longer names the net of U1.5 (GPIO3)
- net LED_1_PIN: no longer names the net of U1.9 (GPIO6)
- net LED_1_PIN: no longer R1.1
- net LED_2_PIN: no longer names the net of U1.10 (GPIO7)
- net LED_3_PIN renamed Reset BTN
- net Reset BTN: now also R3.2, SW1.2
- net LED_READY_PIN: no longer names the net of U1.6 (GPIO4)
- net PWM renamed Player_4
- net Player_4: now also R7.1
- net Power_IN renamed VIN
- net VIN: no longer D1.2 (A)
- new net: D5.2 (A), R7.2
- new net: D2.2 (A), R4.2
- new net: D4.2 (A), R6.2
- new net: D6.2 (A), R8.2
- new net: D3.2 (A), R5.2
- no-connect marks 0 -> 1
Other:
- note added: "Kollane"
- note added: "Punane"
- note added: "Raspberry Pi Pico"
- note added: "Ready Button"
- note added: "Reset Button"
- note added: "Roheline"
- note added: "Sinine"
- note added: "Status LED"
- note added: "User LEDs"
- note added: "Valge"
- note added: "nRF24L01"
- note removed: "Button example"
- note removed: "LED example"
- note removed: "PWM"
- note removed: "Pico W"
- title: Game Server -> Ülemus
- moved on the sheet: BT1, D1, R2, R3, SW1, SW2A, U1

Commit message: skeem update
Other:
- note added: "CE"
- note added: "CSN"
- note added: "GND"
- note added: "IRQ"
- note added: "MISO"
- note added: "MOSI"
- note added: "SCK"
- note added: "VCC"
- moved on the sheet: BT1, SW2A
Changed lines of the file:
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@@
 	(wire
 		(pts
-			(xy 203.2 116.84) (xy 220.98 116.84)
+			(xy 203.2 146.05) (xy 220.98 146.05)
 		)
 		(stroke
@@
 	(wire
 		(pts
-			(xy 248.92 116.84) (xy 256.54 116.84)
+			(xy 248.92 146.05) (xy 256.54 146.05)
 		)
 		(stroke
@@
 	(wire
 		(pts
-			(xy 256.54 116.84) (xy 256.54 123.19)
+			(xy 256.54 146.05) (xy 256.54 152.4)
 		)
 		(stroke
@@
 	(wire
 		(pts
-			(xy 231.14 116.84) (xy 238.76 116.84)
+			(xy 231.14 146.05) (xy 238.76 146.05)
 		)
 		(stroke
@@
 			(width 0)
 			(type default)
+		)
+	)
+	(rectangle
+		(start 205.74 99.06)
+		(end 212.09 102.87)
+		(stroke
+			(width 0)
+			(type default)
+		)
+		(fill
+			(type none)
 		)
 	)
@@
 	)
 	(rectangle
+		(start 205.74 106.68)
+		(end 212.09 110.49)
+		(stroke
+			(width 0)
+			(type default)
+		)
+		(fill
+			(type none)
+		)
+	)
+	(rectangle
+		(start 212.09 106.68)
+		(end 218.44 110.49)
+		(stroke
+			(width 0)
+			(type default)
+		)
+		(fill
+			(type none)
+		)
+	)
+	(rectangle
 		(start 24.13 97.79)
 		(end 81.28 125.73)
+		(stroke
+			(width 0)
+			(type default)
+		)
+		(fill
+			(type none)
+		)
+	)
+	(rectangle
+		(start 205.74 97.79)
+		(end 241.3 115.57)
+		(stroke
+			(width 0)
+			(type default)
+		)
+		(fill
+			(type none)
+		)
+	)
+	(rectangle
+		(start 205.74 102.87)
+		(end 212.09 106.68)
 		(stroke
 			(width 0)
@@
 	)
 	(rectangle
+		(start 212.09 102.87)
+		(end 218.44 106.68)
+		(stroke
+			(width 0)
+			(type default)
+		)
+		(fill
+			(type none)
+		)
+	)
+	(rectangle
 		(start 193.04 31.75)
 		(end 278.13 88.9)
@@
 	)
 	(rectangle
-		(start 193.04 104.14)
-		(end 278.13 130.81)
+		(start 193.04 133.35)
+		(end 278.13 160.02)
+		(stroke
+			(width 0)
+			(type default)
+		)
+		(fill
+			(type none)
+		)
+	)
+	(rectangle
+		(start 212.09 110.49)
+		(end 218.44 114.3)
+		(stroke
+			(width 0)
+			(type default)
+		)
+		(fill
+			(type none)
+		)
+	)
+	(rectangle
+		(start 205.74 110.49)
+		(end 212.09 114.3)
+		(stroke
+			(width 0)
+			(type default)
+		)
+		(fill
+			(type none)
+		)
+	)
+	(rectangle
+		(start 212.09 99.06)
+		(end 218.44 102.87)
 		(stroke
 			(width 0)
@@
 		)
 	)
+	(text "GND"
+		(exclude_from_sim no)
+		(at 208.788 101.346 0)
+		(effects
+			(font
+				(size 1.27 1.27)
+			)
+		)
+	)
+	(text "MOSI"
+		(exclude_from_sim no)
+		(at 215.392 109.22 0)
+		(effects
+			(font
+				(size 1.27 1.27)
+			)
+		)
+	)
 	(text "Valge"
 		(exclude_from_sim no)
@@
 		)
 	)
+	(text "MISO"
+		(exclude_from_sim no)
+		(at 208.788 113.03 0)
+		(effects
+			(font
+				(size 1.27 1.27)
+			)
+		)
+	)
+	(text "CE"
+		(exclude_from_sim no)
+		(at 209.042 105.41 0)
+		(effects
+			(font
+				(size 1.27 1.27)
+			)
+		)
+	)
+	(text "IRQ"
+		(exclude_from_sim no)
+		(at 215.646 113.03 0)
+		(effects
+			(font
+				(size 1.27 1.27)
+			)
+		)
+	)
 	(text "Sinine"
 		(exclude_from_sim no)
@@
 		)
 	)
+	(text "VCC"
+		(exclude_from_sim no)
+		(at 215.392 101.6 0)
+		(effects
+			(font
+				(size 1.27 1.27)
+			)
+		)
+	)
 	(text "User LEDs"
 		(exclude_from_sim no)
@@
 		)
 	)
+	(text "SCK"
+		(exclude_from_sim no)
+		(at 209.042 109.22 0)
+		(effects
+			(font
+				(size 1.27 1.27)
+			)
+		)
+	)
 	(text "Roheline"
 		(exclude_from_sim no)
@@
 		)
 	)
+	(text "CSN"
+		(exclude_from_sim no)
+		(at 215.392 105.41 0)
+		(effects
+			(font
+				(size 1.27 1.27)
+			)
+		)
+	)
 	(text "Kollane"
 		(exclude_from_sim no)
@@
 	(text "Battery"
 		(exclude_from_sim no)
-		(at 194.056 109.728 0)
+		(at 194.056 138.938 0)
 		(effects
 			(font
@@
 	)
 	(label "VIN"
-		(at 203.2 116.84 0)
+		(at 203.2 146.05 0)
 		(fields_autoplaced yes)
 		(effects
@@
 	(symbol
 		(lib_id "Switch:SW_DPST_x2")
-		(at 226.06 116.84 0)
+		(at 226.06 146.05 0)
 		(unit 1)
 		(exclude_from_sim no)
@@
 		(fields_autoplaced yes)
 		(property "Reference" "SW2"
-			(at 226.06 110.49 0)
+			(at 226.06 139.7 0)
 			(effects
 				(font
@@
 		)
 		(property "Value" "SW_DPST_x2"
-			(at 226.06 113.03 0)
+			(at 226.06 142.24 0)
 			(effects
 				(font
@@
 		)
 		(property "Footprint" ""
-			(at 226.06 116.84 0)
+			(at 226.06 146.05 0)
 			(effects
 				(font
@@
 		)
 		(property "Datasheet" "~"
-			(at 226.06 116.84 0)
+			(at 226.06 146.05 0)
 			(effects
 				(font
@@
 		)
 		(property "Description" ""
-			(at 226.06 116.84 0)
+			(at 226.06 146.05 0)
 			(effects
 				(font
@@
 	(symbol
 		(lib_id "power:GND")
-		(at 256.54 123.19 0)
+		(at 256.54 152.4 0)
 		(unit 1)
 		(exclude_from_sim no)
@@
 		(fields_autoplaced yes)
 		(property "Reference" "#PWR03"
-			(at 256.54 129.54 0)
+			(at 256.54 158.75 0)
 			(effects
 				(font
@@
 		)
 		(property "Value" "GND"
-			(at 256.54 128.27 0)
+			(at 256.54 157.48 0)
 			(effects
 				(font
@@
 		)
 		(property "Footprint" ""
-			(at 256.54 123.19 0)
+			(at 256.54 152.4 0)
 			(effects
 				(font
@@
 		)
 		(property "Datasheet" ""
-			(at 256.54 123.19 0)
+			(at 256.54 152.4 0)
 			(effects
 				(font
@@
 		)
 		(property "Description" ""
-			(at 256.54 123.19 0)
+			(at 256.54 152.4 0)
 			(effects
 				(font
@@
 	(symbol
 		(lib_id "Device:Battery")
-		(at 243.84 116.84 90)
+		(at 243.84 146.05 90)
 		(unit 1)
 		(exclude_from_sim no)
@@
 		(fields_autoplaced yes)
 		(property "Reference" "BT1"
-			(at 243.2685 109.22 90)
+			(at 243.2685 138.43 90)
 			(effects
 				(font
@@
 		)
 		(property "Value" "Battery 4xAA"
-			(at 243.2685 111.76 90)
+			(at 243.2685 140.97 90)
 			(effects
 				(font
@@
 		)
 		(property "Footprint" ""
-			(at 242.316 116.84 90)
+			(at 242.316 146.05 90)
 			(effects
 				(font
@@
 		)
 		(property "Datasheet" "~"
-			(at 242.316 116.84 90)
+			(at 242.316 146.05 90)
 			(effects
 				(font
@@
 		)
 		(property "Description" ""
-			(at 243.84 116.84 0)
-			(effects
-				(font
+			(at 243.84 146.05 0)
+			(effects
+				(font

Commit message: eraldi tundub töötavat
Connections:
- net CE: now also U1.29 (GPIO22); no longer U1.22 (GPIO17)
- net CSN: now also U1.22 (GPIO17); no longer U1.21 (GPIO16)
- net MISO: now also U1.21 (GPIO16); no longer U1.26 (GPIO20)
Changed lines of the file:
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@@
 	(title_block
 		(title "Ülemus")
-		(date "2024-11-27")
+		(date "2024-11-29")
 		(comment 1 "Tauno Erik")
 	)
@@
 	(wire
 		(pts
+			(xy 156.21 87.63) (xy 167.64 87.63)
+		)
+		(stroke
+			(width 0)
+			(type default)
+		)
+	)
+	(wire
+		(pts
 			(xy 35.56 111.76) (xy 27.94 111.76)
 		)
@@
 	(wire
 		(pts
+			(xy 156.21 90.17) (xy 167.64 90.17)
+		)
+		(stroke
+			(width 0)
+			(type default)
+		)
+	)
+	(wire
+		(pts
 			(xy 179.07 54.61) (xy 179.07 58.42)
 		)
@@
 	(wire
 		(pts
+			(xy 156.21 95.25) (xy 167.64 95.25)
+		)
+		(stroke
+			(width 0)
+			(type default)
+		)
+	)
+	(wire
+		(pts
 			(xy 156.21 59.69) (xy 163.83 59.69)
 		)
@@
 	(wire
 		(pts
+			(xy 156.21 97.79) (xy 167.64 97.79)
+		)
+		(stroke
+			(width 0)
+			(type default)
+		)
+	)
+	(wire
+		(pts
 			(xy 113.03 97.79) (xy 120.65 97.79)
 		)
@@
 	(wire
 		(pts
+			(xy 156.21 77.47) (xy 167.64 77.47)
+		)
+		(stroke
+			(width 0)
+			(type default)
+		)
+	)
+	(wire
+		(pts
 			(xy 113.03 95.25) (xy 120.65 95.25)
 		)
@@
 	(wire
 		(pts
-			(xy 156.21 90.17) (xy 167.64 90.17)
-		)
-		(stroke
-			(width 0)
-			(type default)
-		)
-	)
-	(wire
-		(pts
 			(xy 214.63 53.34) (xy 224.79 53.34)
 		)
@@
 	(wire
 		(pts
-			(xy 156.21 87.63) (xy 167.64 87.63)
-		)
-		(stroke
-			(width 0)
-			(type default)
-		)
-	)
-	(wire
-		(pts
 			(xy 35.56 59.69) (xy 27.94 59.69)
 		)
@@
 	(wire
 		(pts
-			(xy 156.21 97.79) (xy 167.64 97.79)
-		)
-		(stroke
-			(width 0)
-			(type default)
-		)
-	)
-	(wire
-		(pts
 			(xy 237.49 39.37) (xy 237.49 45.72)
 		)
@@
 	(wire
 		(pts
-			(xy 156.21 95.25) (xy 167.64 95.25)
-		)
-		(stroke
-			(width 0)
-			(type default)
-		)
-	)
-	(wire
-		(pts
 			(xy 27.94 39.37) (xy 27.94 49.53)
-		)
-		(stroke
-			(width 0)
-			(type default)
-		)
-	)
-	(wire
-		(pts
-			(xy 156.21 85.09) (xy 167.64 85.09)
 		)
 		(stroke
@@
 	(global_label "MISO"
 		(shape input)
-		(at 167.64 85.09 0)
+		(at 167.64 97.79 0)
 		(fields_autoplaced yes)
 		(effects
@@
 		)
 		(property "Intersheetrefs" "${INTERSHEET_REFS}"
-			(at 175.2214 85.09 0)
+			(at 175.2214 97.79 0)
 			(effects
 				(font
@@
 	(global_label "CE"
 		(shape input)
+		(at 167.64 77.47 0)
+		(fields_autoplaced yes)
+		(effects
+			(font
+				(size 1.27 1.27)
+			)
+			(justify left)
+		)
+		(property "Intersheetrefs" "${INTERSHEET_REFS}"
+			(at 173.0442 77.47 0)
+			(effects
+				(font
+					(size 1.27 1.27)
+				)
+				(justify left)
+				(hide yes)
+			)
+		)
+	)
+	(global_label "Player_4"
+		(shape input)
+		(at 113.03 95.25 180)
+		(fields_autoplaced yes)
+		(effects
+			(font
+				(size 1.27 1.27)
+			)
+			(justify right)
+		)
+		(property "Intersheetrefs" "${INTERSHEET_REFS}"
+			(at 101.9411 95.25 0)
+			(effects
+				(font
+					(size 1.27 1.27)
+				)
+				(justify right)
+				(hide yes)
+			)
+		)
+	)
+	(global_label "MOSI"
+		(shape input)
+		(at 167.64 87.63 0)
+		(fields_autoplaced yes)
+		(effects
+			(font
+				(size 1.27 1.27)
+			)
+			(justify left)
+		)
+		(property "Intersheetrefs" "${INTERSHEET_REFS}"
+			(at 175.2214 87.63 0)
+			(effects
+				(font
+					(size 1.27 1.27)
+				)
+				(justify left)
+				(hide yes)
+			)
+		)
+	)
+	(global_label "MISO"
+		(shape input)
+		(at 214.63 55.88 180)
+		(fields_autoplaced yes)
+		(effects
+			(font
+				(size 1.27 1.27)
+			)
+			(justify right)
+		)
+		(property "Intersheetrefs" "${INTERSHEET_REFS}"
+			(at 207.0486 55.88 0)
+			(effects
+				(font
+					(size 1.27 1.27)
+				)
+				(justify right)
+				(hide yes)
+			)
+		)
+	)
+	(global_label "CSN"
+		(shape input)
 		(at 167.64 95.25 0)
 		(fields_autoplaced yes)
@@
 		)
 		(property "Intersheetrefs" "${INTERSHEET_REFS}"
-			(at 173.0442 95.25 0)
-			(effects
-				(font
-					(size 1.27 1.27)
-				)
-				(justify left)
-				(hide yes)
-			)
-		)
-	)
-	(global_label "Player_4"
-		(shape input)
-		(at 113.03 95.25 180)
-		(fields_autoplaced yes)
-		(effects
-			(font
-				(size 1.27 1.27)
-			)
-			(justify right)
-		)
-		(property "Intersheetrefs" "${INTERSHEET_REFS}"
-			(at 101.9411 95.25 0)
-			(effects
-				(font
-					(size 1.27 1.27)
-				)
-				(justify right)
-				(hide yes)
-			)
-		)
-	)
-	(global_label "MOSI"
-		(shape input)
-		(at 167.64 87.63 0)
-		(fields_autoplaced yes)
-		(effects
-			(font
-				(size 1.27 1.27)
-			)
-			(justify left)
-		)
-		(property "Intersheetrefs" "${INTERSHEET_REFS}"
-			(at 175.2214 87.63 0)
-			(effects
-				(font
-					(size 1.27 1.27)
-				)
-				(justify left)
-				(hide yes)
-			)
-		)
-	)
-	(global_label "MISO"
-		(shape input)
-		(at 214.63 55.88 180)
-		(fields_autoplaced yes)
-		(effects
-			(font
-				(size 1.27 1.27)
-			)
-			(justify right)
-		)
-		(property "Intersheetrefs" "${INTERSHEET_REFS}"
-			(at 207.0486 55.88 0)
-			(effects
-				(font
-					(size 1.27 1.27)
-				)
-				(justify right)
-				(hide yes)
-			)
-		)
-	)
-	(global_label "CSN"
-		(shape input)
-		(at 167.64 97.79 0)
-		(fields_autoplaced yes)
-		(effects
-			(font
-				(size 1.27 1.27)
-			)
-			(justify left)
-		)
-		(property "Intersheetrefs" "${INTERSHEET_REFS}"
-			(at 174.4352 97.79 0)
-			(effects
-				(font
+			(at 174.4352 95.25 0)
+			(effects
+				(font
